Commit message: feat: redesign robot visuals to look like a research quadruped
Adds cosmetic-only <visual> geometry on top of the existing structural
links: chassis panels/vents/top-cover accent, front camera housing +
lenses, roof lidar puck, IMU cover, status LED, tail light, carry
handle, fastener heads, per-joint QDD pancake motor housings (sized
off each joint's actual torque rating), joint accent rings, leg ribs,
and cable channels. Also unifies the leg tube colors (previously a
grey/green/blue/red mix) into one consistent palette.

None of this touches <collision>, <inertial>, or <joint> — verified
by diff (those blocks are byte-identical to before) and by loading the
regenerated USD in ManagerBasedRLEnv: same 12 revolute + 4 fixed
joints, same joint names, same 48-dim obs / 12-dim action shapes.

File: src/ros2/quadruped_description/urdf/quadruped.urdf (robot description, URDF)
Before this commit: robot quadruped, 17 links, 16 joints
Links:
- link FL_foot_link: geometry collision sphere radius=0.020000; visual cylinder length=0.010000 radius=0.026000
- link FL_hip_link: geometry collision cylinder length=0.062000 radius=0.030000; visual cylinder length=0.004000 radius=0.034000
- link FL_shin_link: geometry collision cylinder length=0.195000 radius=0.016000; visual box size=0.006000 0.010000 0.159900
- link FL_thigh_link: geometry collision cylinder length=0.209000 radius=0.022000; visual box size=0.006000 0.010000 0.171380
- link FR_foot_link: geometry collision sphere radius=0.020000; visual cylinder length=0.010000 radius=0.026000
- link FR_hip_link: geometry collision cylinder length=0.062000 radius=0.030000; visual cylinder length=0.004000 radius=0.034000
- link FR_shin_link: geometry collision cylinder length=0.195000 radius=0.016000; visual box size=0.006000 0.010000 0.159900
- link FR_thigh_link: geometry collision cylinder length=0.209000 radius=0.022000; visual box size=0.006000 0.010000 0.171380
- link RL_foot_link: geometry collision sphere radius=0.020000; visual cylinder length=0.010000 radius=0.026000
- link RL_hip_link: geometry collision cylinder length=0.062000 radius=0.030000; visual cylinder length=0.004000 radius=0.034000
- link RL_shin_link: geometry collision cylinder length=0.195000 radius=0.016000; visual box size=0.006000 0.010000 0.159900
- link RL_thigh_link: geometry collision cylinder length=0.209000 radius=0.022000; visual box size=0.006000 0.010000 0.171380
- link RR_foot_link: geometry collision sphere radius=0.020000; visual cylinder length=0.010000 radius=0.026000
- link RR_hip_link: geometry collision cylinder length=0.062000 radius=0.030000; visual cylinder length=0.004000 radius=0.034000
- link RR_shin_link: geometry collision cylinder length=0.195000 radius=0.016000; visual box size=0.006000 0.010000 0.159900
- link RR_thigh_link: geometry collision cylinder length=0.209000 radius=0.022000; visual box size=0.006000 0.010000 0.171380
- link base_link: geometry collision box size=0.400000 0.200000 0.080000; visual box size=0.012000 0.002000 0.028000
